File: eagle/targetboard.sch (EAGLE design)
At the start: 72 parts, among them CN1 DIP-BLACK-MALE-HEADER-VERT(3P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, IC1 TB6612FNG, IC2 TB6612FNG, IC3 MCP2551, IC4 MCP2551, IC5 LPC1768 or LPC1768, IC6 PMIC-CJT1117-3.3(SOT223), IC7 MAX232D, J1 USB, J2 Serial, J3 CAN, J4 2x8p-2.54, J5 2x8p-2.54, J6 DIP-BLACK-MALE-HEADER-VERT(8P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, J7 2x8p-2.54, Q1 PNP-24V, SW1 SW, Y1 12MHZ

Commit message: Update of board
Parts:
- removed C34, C35, C37, C38: 100nf, Seeed-OPL-Capacitor:CERAMIC-100NF-50V-10%-X7R(0805)
- removed C36: 10uf, Seeed-OPL-Capacitor:CERAMIC-10UF-25V-10%-X5R(0805)
- removed R2, R3: 33.2R, Seeed-OPL-Resistor:SMD-RES-33.2R-1%-1/10W(0603)
- removed R4: 51R, Seeed-OPL-Resistor:SMD-RES-51R-1%-1/10W(0603)
- added C16, C18, C21: 10uf, Seeed-OPL-Capacitor:CERAMIC-10UF-25V-10%-X5R(0805)
- added C19, C20: 100nf, Seeed-OPL-Capacitor:CERAMIC-100NF-50V-10%-X7R(0805)
- added D4: SMD-LED-CLEAR-RED(0805), Seeed-OPL-Diode:SMD-LED-CLEAR-RED(0805)
- added D5: IR 940NM, Seeed-OPL-Diode:DIP-IR-LED-940NM(2P-D5MM)
- added J10: CAN1, Seeed-OPL-Connector:DIP-WHITE-MALE-HEADER-VERT(2P-2.54)
- added J8: 2x8p-2.54, Seeed-OPL-Connector:DIP-BLACK-MALE-HEADER-VERT(2X8P-2.54)
- added J9: CAN2, Seeed-OPL-Connector:DIP-WHITE-MALE-HEADER-VERT(2P-2.54)
- added Q2: NMOSFET, Seeed-OPL-Transistor:SMD-MOSFET-N-CH-60V-300MA-LOGIC-LEVEL-FET(SOT-23)
- added R13: 120R, Seeed-OPL-Resistor:SMD-RES-120R-5%-1/8W(0805)
- added R14: 1.5K, Seeed-OPL-Resistor:SMD-RES-1.5K-1%-1/8W(0805)
- added R15: 100R, Seeed-OPL-Resistor:SMD-RES-100R-5%-1/8W(0805)
- added R16: 2K, Seeed-OPL-Resistor:SMD-RES-2K-5%-1/8W(0805)
- added R17: 390R, Seeed-OPL-Resistor:SMD-RES-390R-5%-1/8W(0805)
- C10, C27: value 10uf -> 100nf; device Seeed-OPL-Capacitor:CERAMIC-10UF-25V-10%-X5R(0805) -> Seeed-OPL-Capacitor:CERAMIC-100NF-50V-10%-X7R(0805)
- C11, C12: value 18pf -> 100nf; device Seeed-OPL-Capacitor:CERAMIC-18PF-50V-5%-NPO(0805) -> Seeed-OPL-Capacitor:CERAMIC-100NF-50V-10%-X7R(0805)
- C13, C4, C5: value 100nf -> 18pf; device Seeed-OPL-Capacitor:CERAMIC-100NF-50V-10%-X7R(0805) -> Seeed-OPL-Capacitor:CERAMIC-18PF-50V-5%-NPO(0805)
- C15: value 18pf -> 10uf; device Seeed-OPL-Capacitor:CERAMIC-18PF-50V-5%-NPO(0805) -> Seeed-OPL-Capacitor:CERAMIC-10UF-10V-10%-X5R(0603)
- C22, C23, C25, C26: value 1uf -> 100nf; device Seeed-OPL-Capacitor:CERAMIC-1UF-25V-10%-X7R(0805) -> Seeed-OPL-Capacitor:CERAMIC-100NF-50V-10%-X7R(0805)
- C24: value 1uf -> 10uf; device Seeed-OPL-Capacitor:CERAMIC-1UF-25V-10%-X7R(0805) -> Seeed-OPL-Capacitor:CERAMIC-10UF-25V-10%-X5R(0805)
- C29, C30, C6: value 100nf -> 1uf; device Seeed-OPL-Capacitor:CERAMIC-100NF-50V-10%-X7R(0805) -> Seeed-OPL-Capacitor:CERAMIC-1UF-25V-10%-X7R(0805)
- C3: value 100nf -> 10uf; device Seeed-OPL-Capacitor:CERAMIC-100NF-50V-10%-X7R(0805) -> Seeed-OPL-Capacitor:CERAMIC-10UF-25V-10%-X5R(0805)
- C31, C32: value 10uf -> 1uf; device Seeed-OPL-Capacitor:CERAMIC-10UF-25V-10%-X5R(0805) -> Seeed-OPL-Capacitor:CERAMIC-1UF-25V-10%-X7R(0805)
- C7: value 10uf -> 100nf; device Seeed-OPL-Capacitor:CERAMIC-10UF-10V-10%-X5R(0603) -> Seeed-OPL-Capacitor:CERAMIC-100NF-50V-10%-X7R(0805)
- IC1: value TB6612FNG -> MCP2551; device Seeed-OPL-ic:DRIVER-TB6612FNG-O/C8/EL(SSOP24) -> Seeed-OPL-ic:INTERFACE-MCP2551-I/SN(SOIC8)
- IC2: value TB6612FNG -> LPC1768 or LPC1768; device Seeed-OPL-ic:DRIVER-TB6612FNG-O/C8/EL(SSOP24) -> Seeed-OPL-ic:MCU_LPC1768FBD100(LQFP100)
- IC3: value MCP2551 -> PMIC-CJT1117-3.3(SOT223); device Seeed-OPL-ic:INTERFACE-MCP2551-I/SN(SOIC8) -> Seeed-OPL-ic:PMIC-CJT1117-3.3(SOT223)
- IC5: value LPC1768 or LPC1768 -> TB6612FNG; device Seeed-OPL-ic:MCU_LPC1768FBD100(LQFP100) -> Seeed-OPL-ic:DRIVER-TB6612FNG-O/C8/EL(SSOP24)
- IC6: value PMIC-CJT1117-3.3(SOT223) -> TB6612FNG; device Seeed-OPL-ic:PMIC-CJT1117-3.3(SOT223) -> Seeed-OPL-ic:DRIVER-TB6612FNG-O/C8/EL(SSOP24)
- J1: value USB -> DIP-BLACK-MALE-HEADER-VERT(8P-2.54); device Seeed-OPL-Connector:MICRO-USB-SMD-TYPE-AB-R/A(ST-USB-001L) -> Seeed-OPL-Connector:DIP-BLACK-MALE-HEADER-VERT(8P-2.54)
- J2: value Serial -> 2x8p-2.54; device Seeed-OPL-Connector:DIP-MALE-DB9-CONNECTOR -> Seeed-OPL-Connector:DIP-BLACK-MALE-HEADER-VERT(2X8P-2.54)
- J3: value CAN -> USB; device Seeed-OPL-Connector:DIP-MALE-DB9-CONNECTOR -> Seeed-OPL-Connector:MICRO-USB-SMD-TYPE-AB-R/A(ST-USB-001L)
- J4: value 2x8p-2.54 -> CAN; device Seeed-OPL-Connector:DIP-BLACK-MALE-HEADER-VERT(2X8P-2.54) -> Seeed-OPL-Connector:DIP-MALE-DB9-CONNECTOR
- J6: value DIP-BLACK-MALE-HEADER-VERT(8P-2.54) -> Serial; device Seeed-OPL-Connector:DIP-BLACK-MALE-HEADER-VERT(8P-2.54) -> Seeed-OPL-Connector:DIP-MALE-DB9-CONNECTOR
- J7: value 2x8p-2.54 -> 2X4P-2.54; device Seeed-OPL-Connector:DIP-BLACK-MALE-HEADER-VERT(2X8P-2.54) -> Seeed-OPL-Connector:DIP-BLACK-FEMALE-HEADER(2X4P-2.54)
- R1, R18: value 1.5K -> 390R; device Seeed-OPL-Resistor:SMD-RES-1.5K-5%-1/16W(0402) -> Seeed-OPL-Resistor:SMD-RES-390R-5%-1/8W(0805)
- R11: value 2K -> 100R; device Seeed-OPL-Resistor:SMD-RES-2K-5%-1/8W(0805) -> Seeed-OPL-Resistor:SMD-RES-100R-5%-1/8W(0805)
- R12: value 2K -> 1.5K; device Seeed-OPL-Resistor:SMD-RES-2K-5%-1/8W(0805) -> Seeed-OPL-Resistor:SMD-RES-1.5K-1%-1/8W(0805)
- R5: value 1.5K -> 51R; device Seeed-OPL-Resistor:SMD-RES-1.5K-5%-1/16W(0402) -> Seeed-OPL-Resistor:SMD-RES-51R-1%-1/10W(0603)
- R6, R7: value 120R -> 33.2R; device Seeed-OPL-Resistor:SMD-RES-120R-5%-1/8W(0805) -> Seeed-OPL-Resistor:SMD-RES-33.2R-1%-1/10W(0603)
- R8: device Seeed-OPL-Resistor:SMD-RES-1.5K-5%-1/16W(0402) -> Seeed-OPL-Resistor:SMD-RES-1.5K-1%-1/8W(0805)
- R9: value 2K -> 120R; device Seeed-OPL-Resistor:SMD-RES-2K-5%-1/8W(0805) -> Seeed-OPL-Resistor:SMD-RES-120R-5%-1/8W(0805)
Connections:
- removed net N$12: IC5.P0.2/TXD0/AD0.7, IC7.DIN1
- removed net N$28: J7.11
- removed net N$29: J7.10
- removed net N$30: J7.9
- removed net N$31: J7.8
- removed net N$32: J7.7
- removed net N$33: J7.6
- new net ESP_0: IC2.P0.4/I2SRX_CLK/CAN_RX2/CAP2.0, J7.2
- new net ESP_2: IC2.P0.5/I2SRX_WS/CAN_TX2/CAP2.1, J7.3
- new net ESP_RST: IC2.P0.6/I2SRX_SDA/SSEL1/MAT2.0, J7.7
- new net IR_SEND: IC2.P1.18/USB_UP/PWM1.1/CAP1.0, Q2.G
- new net N$11: J10.1, R9.1
- new net N$14: D5.+, R11.1
- new net N$21: D5.-, Q2.D
- new net N$24: D4.+, R15.1
- new net RXD0: IC2.P0.3/RXD0/AD0.6, IC7.ROUT1
- new net RX_TO_TX: IC2.P4.29/TX_MCLK/MAT2.1/RXD3, J7.5
- new net TXD0: IC2.P0.2/TXD0/AD0.7, IC7.DIN1
- new net TX_TO_RX: IC2.P4.28/RX_MCLK/MAT2.0/TXD3, J7.1
- net +12V: now also C16.2, C17.1, C23.1, C24.2, IC5.VM1, IC5.VM2, IC5.VM3, IC6.VM1, IC6.VM2, IC6.VM3, J8.1, J8.11; no longer C27.2, C29.1, C31.2, C33.1, IC1.VM1, IC1.VM2, IC1.VM3, IC2.VM1, IC2.VM2, IC2.VM3, J7.16
- net CAN1_H: now also IC1.CANH, J4.7, R9.2; no longer IC4.CANH, J3.7, R6.2
- net CAN1_L: now also IC1.CANL, J10.2, J4.2; no longer IC4.CANL, J3.2, R6.1
- net CAN1_REF: now also IC1.VREF, IC2.P1.27/CLKOUT/USB_OVRCR/CAP0.1; no longer IC4.VREF, IC5.P1.27/CLKOUT/USB_OVRCR/CAP0.1
- net CAN1_RS: now also IC1.RS, IC2.P1.26/MC1B/PWM1.6/CAP0.0; no longer IC4.RS, IC5.P1.26/MC1B/PWM1.6/CAP0.0
- net CAN1_RX: now also IC1.RXD, IC2.P0.1/CAN_TX1/RXD3/SCL1, J8.8; no longer IC4.RXD, IC5.P0.1/CAN_TX1/RXD3/SCL1
- net CAN1_TX: now also IC1.TXD, IC2.P0.0/CAN_RX1/TXD3/SDA1; no longer IC4.TXD, IC5.P0.0/CAN_RX1/TXD3/SDA1
- net CAN2_H: now also IC4.CANH, J4.8, R13.2; no longer IC3.CANH, J3.8, R7.2
- net CAN2_L: now also IC4.CANL, J4.1, J9.2; no longer IC3.CANL, J3.1, R7.1
- net CAN2_REF: now also IC2.P2.3/PWM1.4/DCD1/TRACEDATA2, IC4.VREF; no longer IC3.VREF, IC5.P2.3/PWM1.4/DCD1/TRACEDATA2
- net CAN2_RS: now also IC2.P2.6/PCAP1.0/RI1/TRACECLK, IC4.RS; no longer IC3.RS, IC5.P2.6/PCAP1.0/RI1/TRACECLK
- net CAN2_RX: now also IC2.P2.7/CAN_RX2/RTS1, IC4.RXD, J8.9; no longer IC3.RXD, IC5.P2.7/CAN_RX2/RTS1
- net CAN2_TX: now also IC2.P2.8/CAN_TX2/TXD2, IC4.TXD; no longer IC3.TXD, IC5.P2.8/CAN_TX2/TXD2
- net CM1A: now also IC2.P1.9/ENET_RXD0, IC6.ATN2; no longer IC2.ATN2, IC5.P1.9/ENET_RXD0
- net CM1B: now also IC2.P1.8/ENET_CRS, IC6.ATN1; no longer IC2.ATN1, IC5.P1.8/ENET_CRS
- net CM2A: now also IC2.P1.1/ENET-TXD1, IC6.BIN1; no longer IC2.BIN1, IC5.P1.1/ENET-TXD1
- net CM2B: now also IC2.P1.0/ENET-TXD0, IC6.BIN2; no longer IC2.BIN2, IC5.P1.0/ENET-TXD0
- net CM3A: now also IC2.P0.9/I2STX_SDA/MOSI1/MAT2.3, IC5.ATN2; no longer IC1.ATN2, IC5.P0.9/I2STX_SDA/MOSI1/MAT2.3
- net CM3B: now also IC2.P1.10/ENET_RXD1, IC5.ATN1; no longer IC1.ATN1, IC5.P1.10/ENET_RXD1
- net CM4A: now also IC2.P1.14/ENET-RX_ER, IC5.BIN1; no longer IC1.BIN1, IC5.P1.14/ENET-RX_ER
- net CM4B: now also IC2.P0.8/I2STX_WS/MISO1/MAT2.2, IC5.BIN2; no longer IC1.BIN2, IC5.P0.8/I2STX_WS/MISO1/MAT2.2
- net DM: now also J3.DM, R6.2; no longer J1.DM, R3.2
- net DP: now also J3.DP, R7.2, R8.1; no longer J1.DP, R1.1, R2.2
- net EDM: now also C5.2, IC2.P0.30/USB_D-, R6.1; no longer C14.2, IC5.P0.30/USB_D-, R3.1
- net EDP: now also C4.2, IC2.P0.29/USB_D+, R7.1; no longer C15.2, IC5.P0.29/USB_D+, R2.1
- net GND: now also C10.2, C13.1, C16.1, C18.1, C19.1, C20.1, C21.1, C22.1, C23.2, C24.1, C26.2, C29.1, C31.2, C33.1, C6.2, C7.2, C8.2, C9.2, D4.-, IC1.VDD, IC2.RTCX1, IC2.VREFN, IC2.VSS@1, IC2.VSS@2, IC2.VSS@3, IC2.VSS@4, IC2.VSS@5, IC2.VSS@6, IC2.VSSA, IC3.GND, IC5.GND, IC5.PGND, IC5.PGND2, IC5.PGND2@1, IC5.PGND@1, IC6.PGND, IC6.PGND2, IC6.PGND2@1, IC6.PGND@1, J2.10, J2.11, J2.12, J2.13, J2.14, J2.15, J2.9, J3.GND, J3.GND@1, J3.GND@2, J4.3, J4.5, J4.6, J6.5, J7.4, J8.16, J8.7, Q2.S; no longer C10.1, C13.2, C24.2, C26.1, C29.2, C30.2, C31.1, C32.1, C33.2, C34.2, C35.1, C36.1, C37.2, C38.2, C6.1, C7.1, C8.1, C9.1, IC1.GND, IC1.PGND, IC1.PGND2, IC1.PGND2@1, IC1.PGND@1, IC2.GND, IC2.PGND, IC2.PGND2, IC2.PGND2@1, IC2.PGND@1, IC3.VDD, IC5.VREFN, IC5.VSS@1, IC5.VSS@2, IC5.VSS@3, IC5.VSS@4, IC5.VSS@5, IC5.VSS@6, IC5.VSSA, J1.GND, J2.5, J2.7, J3.10, J3.11, J3.3, J3.5, J3.6, J4.12, J4.13, J4.14, J4.15, J4.9, J7.1
- net IR_IN: now also IC2.P0.24/AD0.1/I2SRX_WS/CAP3.1; no longer IC5.P0.24/AD0.1/I2SRX_WS/CAP3.1
- net LED1: now also IC2.P0.23/AD0.0/I2SRX_CLK/CAP3.0, R1.1; no longer IC5.P0.27/SDA0/USB_SDA, R9.1
- net LED2: now also IC2.P3.25/MAT0.0/PWM1.2, R17.1; no longer IC5.P3.25/MAT0.0/PWM1.2, R11.1
- net LED3: now also IC2.P3.26/STCLK/MAT0.1/PWM1.3, R18.1; no longer IC5.P3.26/STCLK/MAT0.1/PWM1.3, R12.1
- net M1A: now also IC6.AO1, IC6.AO@1, J8.2; no longer IC2.AO1, IC2.AO@1, J7.2
- net M1B: now also IC6.AO2, IC6.AO2@1, J8.15; no longer IC2.AO2, IC2.AO2@1, J7.15
- net M2A: now also IC6.BO2, IC6.BO2@1, J8.3; no longer IC2.BO2, IC2.BO2@1, J7.3
- net M2B: now also IC6.BO1, IC6.BO1@1, J8.14; no longer IC2.BO1, IC2.BO1@1, J7.14
- net M3A: now also IC5.AO1, IC5.AO@1, J8.4; no longer IC1.AO1, IC1.AO@1, J7.4
- net M3B: now also IC5.AO2, IC5.AO2@1, J8.13; no longer IC1.AO2, IC1.AO2@1, J7.13
- net M4A: now also IC5.BO2, IC5.BO2@1, J8.5; no longer IC1.BO2, IC1.BO2@1, J7.5
- net M4B: now also IC5.BO1, IC5.BO1@1, J8.12; no longer IC1.BO1, IC1.BO1@1, J7.12
- net N$1: now also IC2.P0.10/TXD2/SDA2/MAT3.0, J1.1, J2.1, J2.16; no longer IC5.P0.10/TXD2/SDA2/MAT3.0, J5.1, J5.16, J6.1
- net N$10: now also IC2.P1.30/VBUS/AD0.4, R14.2; no longer IC5.P1.30/VBUS/AD0.4, R5.1
- net N$13: now also J9.1, R13.1; no longer IC5.P0.3/RXD0/AD0.6, IC7.ROUT1
- net N$15: now also C30.2; no longer C23.2
- net N$16: now also C30.1; no longer C23.1
- net N$17: now also C32.1; no longer C22.1
- net N$18: now also C32.2; no longer C22.2
- net N$19: now also C29.2; no longer C26.2
- net N$2: now also IC2.P2.10/EINT0N/NMI, R12.1; no longer IC5.P2.10/EINT0N/NMI, R8.1
- net N$20: now also C31.1; no longer C25.1
- net N$22: now also IC2.P0.18/DCD1/MOSI0/MOSI1; no longer IC5.P0.18/DCD1/MOSI0/MOSI1
- net N$3: now also R18.2; no longer R12.2
- net N$4: now also R17.2; no longer R11.2
- net N$5: now also R1.2; no longer R9.2
- net N$6: now also C14.2, IC2.X1; no longer C12.2, IC5.X1
- net N$7: now also R8.2; no longer R1.2
- net N$8: now also C13.2, IC2.X2; no longer C11.2, IC5.X2
- net N$9: now also R5.2; no longer R4.2
- net NTRST: now also IC2.TRST_N, J5.2; no longer IC5.TRST_N, J4.2
- net P2_9: now also IC2.P2.9/USB_CONNECT/RXD2, R5.1; no longer IC5.P2.9/USB_CONNECT/RXD2, R4.1
- net PWM1: now also IC2.P2.4/PWM1.5/DSR1/TRACEDATA1, IC6.PWMA; no longer IC2.PWMA, IC5.P2.4/PWM1.5/DSR1/TRACEDATA1
- net PWM2: now also IC2.P2.5/PWM1.6/DTR1/TRACEDATA0, IC6.PWMB; no longer IC2.PWMB, IC5.P2.5/PWM1.6/DTR1/TRACEDATA0
- net PWM3: now also IC2.P1.21/MCABORT/PWM1.3/SSEL0, IC5.PWMA; no longer IC1.PWMA, IC5.P1.21/MCABORT/PWM1.3/SSEL0
- net PWM4: now also IC2.P1.23/MCFB1/PWM1.4/MISO0, IC5.PWMB; no longer IC1.PWMB, IC5.P1.23/MCFB1/PWM1.4/MISO0
- net RST: now also IC2.NRESET, J5.8, R16.1; no longer IC5.NRESET, J4.8, R18.1
- net RTCK: now also IC2.RTCK, J5.6; no longer IC5.RTCK, J4.6
- net RX3: now also IC2.P0.26/AD0.3/AOUT/RXD3; no longer IC5.P0.26/AD0.3/AOUT/RXD3
- net RXD1: now also IC2.P2.1/PWM1.2/RXD1; no longer IC5.P2.1/PWM1.2/RXD1
- net SER1_RX: now also J6.2; no longer J2.2
- net SER1_TX: now also J6.3; no longer J2.3
- net SER2_RX: now also J6.1; no longer J2.1
- net SER2_TX: now also J6.6; no longer J2.6
- net STBY: now also IC2.P1.4/ENET-TX_EN, IC5.STBY, IC6.STBY; no longer IC1.STBY, IC2.STBY, IC5.P1.4/ENET-TX_EN
- net TCK: now also IC2.TCK/SWDCLK, J5.5; no longer IC5.TCK/SWDCLK, J4.5
- net TDI: now also IC2.TDI, J5.3; no longer IC5.TDI, J4.3
- net TDO: now also IC2.TDO/SWO, J5.7; no longer IC5.TDO/SWO, J4.7
- net TMS: now also IC2.TMS/SWDIO, J5.4; no longer IC5.TMS/SWDIO, J4.4
- net TX3: now also IC2.P0.25/AD0.2/I2SRX_SDA/TXD3; no longer IC5.P0.25/AD0.2/I2SRX_SDA/TXD3
- net TXD1: now also IC2.P2.0/PWM1.1/TXD1/TRACECLK; no longer IC5.P2.0/PWM1.1/TXD1/TRACECLK
- net T_RTCK: now also IC2.P0.21/RI1/CAN_RX1, J1.6, J2.6; no longer IC5.P0.21/RI1/CAN_RX1, J5.6, J6.6
- net T_SRST: now also IC2.P0.22/RTS1/CAN_TX1, J1.8, J2.8; no longer IC5.P0.22/RTS1/CAN_TX1, J5.8, J6.8
- net T_SWDCLK: now also IC2.P0.15/TXD1/SCK0/SCK, J1.5, J2.5; no longer IC5.P0.15/TXD1/SCK0/SCK, J5.5, J6.5
- net T_SWDIO: now also IC2.P0.17/CTS1/MISO0/MISO, J1.4, J2.4; no longer IC5.P0.17/CTS1/MISO0/MISO, J5.4, J6.4
- net T_SWO: now also IC2.P0.11/RXD2/SCL2/MAT3.1, J1.7, J2.7; no longer IC5.P0.11/RXD2/SCL2/MAT3.1, J5.7, J6.7
- net T_TDI: now also IC2.P0.20/DTR1/SCL1, J1.3, J2.3; no longer IC5.P0.20/DTR1/SCL1, J5.3, J6.3
- net T_TRST: now also IC2.P0.16/RXD1/SSEL0/SSEL, J1.2, J2.2; no longer IC5.P0.16/RXD1/SSEL0/SSEL, J5.2, J6.2
- net VCC: now also C15.2, C33.2, C6.1, C7.1, C8.1, IC1.VSS, IC3.IN, J3.VCC, J8.6, R11.2, R14.1; no longer C17.1, C24.1, C35.2, C37.1, C7.2, IC3.VSS, IC6.IN, J1.VCC, R5.2
- net VDD: now also C10.1, C11.2, C12.2, C18.2, C19.2, C20.2, C21.2, C22.2, C25.1, C26.1, C27.2, C9.1, IC2.VBAT, IC2.VDD3.3V@1, IC2.VDD3.3V@2, IC2.VDD3.3V@3, IC2.VDD3.3V@4, IC2.VDDA, IC2.VDDREG3.3V@1, IC2.VDDREG3.3V@2, IC2.VREFP, IC3.OUT, IC5.VCC, IC6.VCC, J5.1, J5.16, J7.6, J7.8, J8.10, R12.2, R15.2, R16.2; no longer C10.2, C13.1, C30.1, C32.2, C34.1, C36.2, C38.1, C4.2, C5.2, C6.2, C8.2, C9.2, IC1.VCC, IC2.VCC, IC5.VBAT, IC5.VDD3.3V@1, IC5.VDD3.3V@2, IC5.VDD3.3V@3, IC5.VDD3.3V@4, IC5.VDDA, IC5.VDDREG3.3V@1, IC5.VDDREG3.3V@2, IC5.VREFP, IC6.OUT, J4.1, J4.16, R18.2, R8.2
Other:
- moved on the sheet: C1, C10, C11, C12, C13, C14, C15, C17, C2, C22, C23, C24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
